File: hardware/adc.sch (KiCad schematic (older format))
At the start: 38 parts, among them U39 LP5907-3.0, U8 LTC2292

Commit message: Update kicad:  * kicad_pcb from 20170123 to 20171130 (pcbnew from 75cda50 to 5ecfd32)  * EESchema from 2 to 4
fix pin 53 in U33 (remove path in pcb)
Parts:
- C163, C164, C165, C166, C167, C168, C19, C20, C216, C217, C218, C219, C22, C220, C221, C222, C223, C224, C225, C23, C24, C248, C249, C25, C27, C30, C31: symbol C -> Device:C
- R100, R20, R21, R91, R92, R93, R97, R98, R99: symbol R -> Device:R
- U39: symbol LP5907 -> fmcw3:LP5907
- U8: footprint Housings_DFN_QFN:QFN-64-1EP_9x9mm_Pitch0.5mm -> Package_DFN_QFN:QFN-64-1EP_9x9mm_P0.5mm_EP7.35x7.35mm; symbol LTC229X -> fmcw3:LTC229X
