File: hardware/if.sch (KiCad schematic (older format))
At the start: 59 parts, among them U34 ADA4940-2, U35 ADA4940-2

Commit message: Update kicad:  * kicad_pcb from 20170123 to 20171130 (pcbnew from 75cda50 to 5ecfd32)  * EESchema from 2 to 4
fix pin 53 in U33 (remove path in pcb)
Parts:
- C124, C125, C126, C127, C128, C129, C130, C131, C132, C133, C134, C135, C136, C137, C138, C139, C140, C141, C142, C143, C144, C145, C146, C147, C148, C149, C150, C151, C173: symbol C -> Device:C
- L10, L11, L8, L9: symbol INDUCTOR_SMALL -> Device:L_Small
- R55, R56, R57, R58, R59, R60, R61, R62, R63, R64, R65, R66, R67, R68, R74, R75, R76, R77, R78, R86, R87, R89, R90, R94: symbol R -> Device:R
- U34, U35: symbol ADA4940-2 -> fmcw3:ADA4940-2
Connections:
- wire segments 164 -> 217
