File: hardware/mixer.sch (KiCad schematic (older format))
At the start: 31 parts, among them U26 5400BL15B050E, U27 5400BL15B050E, U28 5400BL15B050E, U29 ADL5802

Commit message: Update kicad:  * kicad_pcb from 20170123 to 20171130 (pcbnew from 75cda50 to 5ecfd32)  * EESchema from 2 to 4
fix pin 53 in U33 (remove path in pcb)
Parts:
- C107, C108, C109, C110, C111, C112, C113, C114, C115, C116, C117, C118, C119, C120, C121, C122, C123, C162: symbol C -> Device:C
- F1, F2: symbol Via -> fmcw3:Via
- FB13: symbol FILTER -> Device:L_Core_Ferrite
- R49, R50, R51, R52, R53, R54: symbol R -> Device:R
- U26, U27, U28: symbol 5400BL15B050E -> fmcw3:5400BL15B050E
- U29: footprint Housings_DFN_QFN:QFN-24-1EP_4x4mm_Pitch0.5mm -> Package_DFN_QFN:QFN-24-1EP_4x4mm_P0.5mm_EP2.6x2.6mm; symbol ADL5802 -> fmcw3:ADL5802
Connections:
- wire segments 91 -> 122
