File: hardware/power.sch (KiCad schematic (older format))
At the start: 96 parts, among them CON2 BARREL_JACK, U17 L7980, U18 L7980, U19 L7980, U20 LP5907-3.0, U21 LP2985A-10DBVR, U22 TPS7A91, U23 TPS7A91, U24 TPS7A91, U25 MIC5301-3.3

Commit message: Update kicad:  * kicad_pcb from 20170123 to 20171130 (pcbnew from 75cda50 to 5ecfd32)  * EESchema from 2 to 4
fix pin 53 in U33 (remove path in pcb)
Parts:
- C100, C101, C102, C103, C104, C105, C106, C169, C172, C175, C177, C178, C60, C61, C62, C63, C64, C65, C66, C67, C68, C69, C70, C71, C72, C73, C74, C75, C76, C77, C78, C79, C80, C81, C82, C83, C84, C85, C86, C87, C88, C89, C90, C91, C92, C93, C94, C95, C96, C97, C98, C99: symbol C -> Device:C
- CON2: value BARREL_JACK -> Barrel_Jack; symbol BARREL_JACK -> Connector_Specialized:Barrel_Jack
- D1: symbol LED -> Device:LED_ALT
- D2, D3, D4: symbol D_Schottky -> Device:D_Schottky
- FB11: symbol FILTER -> Device:L_Core_Ferrite
- L5, L6, L7: symbol INDUCTOR_SMALL -> Device:L_Small
- R101, R103, R104, R24, R25, R26, R27, R28, R29, R30, R31, R32, R33, R34, R35, R36, R37, R38, R41, R42, R43, R44, R45, R46, R47, R48: symbol R -> Device:R
- U17, U18, U19: footprint Housings_DFN_QFN:DFN-8-1EP_3x3mm_Pitch0.5mm -> Package_DFN_QFN:DFN-8-1EP_3x3mm_P0.5mm_EP1.66x2.38mm; symbol L7981 -> fmcw3:L7981
- U20: symbol LP5907 -> fmcw3:LP5907
- U21: symbol LP2985 -> fmcw3:LP2985
- U22, U23, U24: symbol TPS7A91 -> fmcw3:TPS7A91
- U25: symbol MIC5301 -> fmcw3:MIC5301
Connections:
- wire segments 182 -> 264
