File: hardware/rx.sch (KiCad schematic (older format))
At the start: 19 parts, among them P1 SMA, U11 SKY65404, U9 TRF37A73

Commit message: Update kicad:  * kicad_pcb from 20170123 to 20171130 (pcbnew from 75cda50 to 5ecfd32)  * EESchema from 2 to 4
fix pin 53 in U33 (remove path in pcb)
Parts:
- C179, C180, C35, C42, C44, C46, C47, C48, C49, C50, C54: symbol C -> Device:C
- FB7, FB8: symbol FILTER -> Device:L_Core_Ferrite
- L1, L2: symbol INDUCTOR -> Device:L
- P1: symbol SMA -> fmcw3:SMA
- R22: symbol R -> Device:R
- U11: symbol SKY65404 -> fmcw3:SKY65404
- U9: symbol TRF37A75 -> fmcw3:TRF37A75
Connections:
- wire segments 39 -> 54
Changed lines of the file:
@@
-EESchema Schematic File Version 2
+EESchema Schematic File Version 4
 LIBS:power
-LIBS:device
-LIBS:transistors
-LIBS:conn
-LIBS:linear
-LIBS:regul
-LIBS:74xx
-LIBS:cmos4000
-LIBS:adc-dac
-LIBS:memory
-LIBS:xilinx
-LIBS:microcontrollers
-LIBS:dsp
-LIBS:microchip
-LIBS:analog_switches
-LIBS:motorola
-LIBS:texas
-LIBS:intel
-LIBS:audio
-LIBS:interface
-LIBS:digital-audio
-LIBS:philips
-LIBS:display
-LIBS:cypress
-LIBS:siliconi
-LIBS:opto
-LIBS:atmel
-LIBS:contrib
-LIBS:valves
+LIBS:Device
+LIBS:Connector_Specialized
+LIBS:Connector_Generic
+LIBS:Logic_74xgxx
+LIBS:Logic_CMOS_4000
+LIBS:Valve
 LIBS:fmcw3
-LIBS:fmcw3-cache
+LIBS:Switch
 EELAYER 26 0
 EELAYER END
@@
 $EndDescr
 $Comp
-L SKY65404 U11
+L fmcw3:SKY65404 U11
 U 1 1 593BC199
 P 6800 3800
@@
 $EndComp
 $Comp
-L GND #PWR0122
+L power:GND #PWR0122
 U 1 1 593BC25F
 P 6850 4350
@@
 $EndComp
 $Comp
-L GND #PWR0123
+L power:GND #PWR0123
 U 1 1 593BC2B3
 P 8000 4200
@@
 	8000 3800 8000 4200
 $Comp
-L GND #PWR0124
+L power:GND #PWR0124
 U 1 1 593BC302
 P 5900 4350
@@
 	5900 3800 5900 4350
 $Comp
-L R R22
+L Device:R R22
 U 1 1 593BC396
 P 5750 3650
@@
 Wire Wire Line
 	7600 3650 7600 3300
-Wire Wire Line
-	7600 3300 7850 3300
-$Comp
-L INDUCTOR L2
+$Comp
+L Device:L L2
 U 1 1 593BC695
 P 8150 3300
 AR Path="/59396B97/593BC695" Ref="L2"  Part="1"
 AR Path="/593D90BA/593BC695" Ref="L4"  Part="1"
+AR Path="/593BC695" Ref="L4"  Part="1"
 F 0 "L4" V 8100 3300 50  0000 C CNN
 F 1 "0.6n" V 8250 3300 50  0000 C CNN
@@
 $EndComp
 $Comp
-L C C49
+L Device:C C49
 U 1 1 593BC767
 P 8600 3450
@@
 	1    0    0    -1
 $EndComp
-Wire Wire Line
-	8600 3300 8450 3300
-$Comp
-L GND #PWR0125
+$Comp
+L power:GND #PWR0125
 U 1 1 593BC7DB
 P 8600 3600
@@
 $EndComp
 Wire Wire Line
-	7600 3950 8950 3950
-$Comp
-L SMA P1
+	7600 3950 8450 3950
+$Comp
+L fmcw3:SMA P1
 U 1 1 593BCCCA
 P 9150 3950
@@
 $EndComp
 $Comp
-L GND #PWR0126
+L power:GND #PWR0126
 U 1 1 593BCD59
 P 9150 4100
@@
 $EndComp
 $Comp
-L C C48
+L Device:C C48
 U 1 1 593BCEBC
 P 8450 4200
@@
 Connection ~ 8450 3950
 $Comp
-L GND #PWR0127
+L power:GND #PWR0127
 U 1 1 593BCF37
 P 8450 4350
@@
 	6100 3950 5700 3950
 $Comp
-L C C46
+L Device:C C46
 U 1 1 593BD4EF
 P 5550 3950
@@
 	5400 3950 5100 3950
 $Comp
-L GND #PWR0128
+L power:GND #PWR0128
 U 1 1 593BD727
 P 4350 4850
@@
 $EndComp
 Wire Wire Line
-	4350 4600 4350 4850
-$Comp
-L INDUCTOR L1
+	4350 4600 4350 4700
+$Comp
+L Device:L L1
 U 1 1 593BD8E8
 P 3850 3750
 AR Path="/59396B97/593BD8E8" Ref="L1"  Part="1"
 AR Path="/593D90BA/593BD8E8" Ref="L3"  Part="1"
+AR Path="/593BD8E8" Ref="L3"  Part="1"
 F 0 "L3" V 3800 3750 50  0000 C CNN
-F 1 "LQW15AN9N9J80D" V 3950 3750 50  0000 C CNN
+F 1 "LQW15AN9N9J80D" V 3950 3700 50  0000 C CNN
 F 2 "fmcw3:C_0402b" H 3850 3750 60  0001 C CNN
 F 3 "" H 3850 3750 60  0000 C CNN
@@
 $EndComp
 Wire Wire Line
-	3600 4050 4000 4050
+	3600 4050 3850 4050
 Connection ~ 3850 4050
 $Comp
-L C C44
+L Device:C C44
 U 1 1 593BDA25
 P 4050 3250
@@
 $EndComp
 Wire Wire Line
-	3850 3100 4300 3100
-Wire Wire Line
-	3850 2700 3850 3450
-$Comp
-L GND #PWR0129
+	3850 3100 4050 3100
+Wire Wire Line
+	3850 2700 3850 2750
+$Comp
+L power:GND #PWR0129
 U 1 1 593BDABD
 P 4050 3400
@@
 Connection ~ 3850 3100
 $Comp
-L C C42
+L Device:C C42
 U 1 1 593BDF98
 P 3450 4050
@@
 	3300 4050 3150 4050
 Wire Wire Line
-	8600 2600 8600 3300
+	8600 2600 8600 3100
 Text HLabel 2850 2750 0    60   Input ~ 0
 3V0
-Wire Wire Line
-	3650 2750 3850 2750
 Text HLabel 7500 2600 0    60   Input ~ 0
 3V0
-Wire Wire Line
-	8500 2600 9100 2600
 Text HLabel 3150 4050 0    60   Output ~ 0
 RF_OUT
@@
 15 mA
 $Comp
-L FILTER FB7
+L Device:L_Core_Ferrite FB7
 U 1 1 59751767
 P 3300 2750
 AR Path="/593D90BA/59751767" Ref="FB7"  Part="1"
 AR Path="/59396B97/59751767" Ref="FB5"  Part="1"
-F 0 "FB7" H 3300 2900 50  0000 C CNN
-F 1 "BLM18PG181SN1D" H 3300 2650 50  0000 C CNN
+AR Path="/59751767" Ref="FB7"  Part="1"
+F 0 "FB7" V 3400 2750 50  0000 C CNN
+F 1 "BLM18PG181SN1D" V 3250 2750 50  0000 C CNN
 F 2 "fmcw3:C_0603b" H 3300 2750 60  0001 C CNN
 F 3 "" H 3300 2750 60  0000 C CNN
 	1    3300 2750
-	1    0    0    -1
-$EndComp
-Wire Wire Line
-	2850 2750 2950 2750
-$Comp
-L C C54
+	0    -1   -1   0
+$EndComp
+Wire Wire Line
+	2850 2750 2900 2750
+$Comp
+L Device:C C54
 U 1 1 59751D28
 P 5000 2900
@@
 $EndComp
 $Comp
-L GND #PWR0142
+L power:GND #PWR0142
 U 1 1 59751D9B
 P 5000 3050
@@
 Connection ~ 3850 2750
 $Comp
-L C C35
+L Device:C C35
 U 1 1 59752286
 P 2900 3000
@@
 $EndComp
 $Comp
-L GND #PWR0143
+L power:GND #PWR0143
 U 1 1 59752325
 P 2900 3150
@@
 Connection ~ 2900 2750
 $Comp
-L FILTER FB8
+L Device:L_Core_Ferrite FB8
 U 1 1 597527FA
 P 8150 2600
 AR Path="/593D90BA/597527FA" Ref="FB8"  Part="1"
 AR Path="/59396B97/597527FA" Ref="FB6"  Part="1"
-F 0 "FB8" H 8150 2750 50  0000 C CNN
-F 1 "BLM18PG181SN1D" H 8150 2500 50  0000 C CNN
+AR Path="/597527FA" Ref="FB8"  Part="1"
+F 0 "FB8" V 8250 2600 50  0000 C CNN
+F 1 "BLM18PG181SN1D" V 8100 2600 50  0000 C CNN
 F 2 "fmcw3:C_0603b" H 8150 2600 60  0001 C CNN
 F 3 "" H 8150 2600 60  0000 C CNN
 	1    8150 2600
-	1    0    0    -1
-$EndComp
-Wire Wire Line
-	7500 2600 7800 2600
-$Comp
-L C C50
+	0    -1   -1   0
+$EndComp
+Wire Wire Line
+	7500 2600 7550 2600
+$Comp
+L Device:C C50
 U 1 1 59752C43
 P 9100 2750
@@
 $EndComp
 $Comp
-L GND #PWR0132
+L power:GND #PWR0132
 U 1 1 59752C49
 P 9100 2900
@@
 $EndComp
 $Comp
-L C C47
+L Device:C C47
 U 1 1 59752CDE
 P 7550 2800
@@
 $EndComp
 $Comp
-L GND #PWR0133
+L power:GND #PWR0133
 U 1 1 59752CE4
 P 7550 2950
@@
 Gain: 11 dB\nNF: 5.5 dB\nIP1dB: -3 dBm
 $Comp
-L TRF37A75 U9
+L fmcw3:TRF37A75 U9
 U 1 1 597605DF
 P 4550 4100
@@
 	4750 4700 4750 4600
 Wire Wire Line
-	4350 4700 4750 4700
+	4350 4700 4450 4700
 Wire Wire Line
 	4650 4700 4650 4600
@@
 Connection ~ 4350 4700
 $Comp
-L C C180
+L Device:C C180
 U 1 1 59761DBE
 P 4700 3100
@@
 $EndComp
 $Comp
-L GND #PWR0247
+L power:GND #PWR0247
 U 1 1 59761E7D
 P 4700 3250
@@
 	5000 2750 5000 2700
 $Comp
-L C C179
+L Device:C C179
 U 1 1 59762FC5
 P 4300 3250
@@
 Connection ~ 4050 3100
 $Comp
-L GND #PWR0248
+L power:GND #PWR0248
 U 1 1 5976305E
 P 4300 3400
@@
 	5200 4100 5200 4250
 $Comp
-L GND #PWR0252
+L power:GND #PWR0252
 U 1 1 59765731
 P 5200 4250
@@
 $EndComp
 Wire Wire Line
-	5000 2700 3850 2700
+	5000 2700 4700 2700
 Text Notes 5700 2200 0    60   ~ 0
 Gain: 26 dB\nIP1dB: -16 dBm
+Wire Wire Line
+	3850 4050 3850 3900
+Wire Wire Line
+	8450 3950 8950 3950
+Wire Wire Line
+	3850 4050 4000 4050
+Wire Wire Line
+	3850 2750 3850 3100
+Wire Wire Line
+	8600 2600 9100 2600
+Wire Wire Line
+	8600 3100 8600 3300
+Wire Wire Line
+	4650 4700 4750 4700
+Wire Wire Line
+	4550 4700 4650 4700
+Wire Wire Line
+	4450 4700 4550 4700
+Wire Wire Line
+	4350 4700 4350 4850
+Wire Wire Line
+	4700 2700 3850 2700
+Wire Wire Line
+	4050 3100 4300 3100
+Wire Wire Line
+	3850 3100 3850 3600
+Wire Wire Line
+	8300 3300 8600 3300
+Wire Wire Line
+	7600 3300 8000 3300
+Wire Wire Line
+	3450 2750 3850 2750
+Wire Wire Line
+	2900 2750 3150 2750
+Wire Wire Line
+	8300 2600 8600 2600
+Wire Wire Line
+	7550 2600 8000 2600
 $EndSCHEMATC
