File: hardware/tx.sch (KiCad schematic (older format))
At the start: 54 parts, among them Q1 RE1C002UN, U1 ADF4158, U10 HMC431LP4, U12 PAT1220-6dB, U14 MGA-25203, U15 SMA, U3 PAT1220-6dB, U7 TLV172DCK

Commit message: Update kicad:  * kicad_pcb from 20170123 to 20171130 (pcbnew from 75cda50 to 5ecfd32)  * EESchema from 2 to 4
fix pin 53 in U33 (remove path in pcb)
Parts:
- C10, C11, C14, C176, C2, C21, C214, C215, C26, C28, C29, C3, C32, C33, C34, C36, C37, C38, C39, C4, C40, C41, C43, C5, C6, C7, C8: symbol C -> Device:C
- FB2, FB3, FB4: symbol FILTER -> Device:L_Core_Ferrite
- Q1: symbol MOS_N_GSD -> fmcw3:MOS_N_GSD
- R1, R10, R11, R12, R14, R17, R18, R2, R39, R4, R40, R5, R6, R7, R9: symbol R -> Device:R
- U1: symbol ADF4158 -> fmcw3:ADF4158
- U10: symbol HMC431LP4 -> fmcw3:HMC431LP4
- U12, U3: symbol PAT1220 -> fmcw3:PAT1220
- U14: symbol MGA-25203 -> fmcw3:MGA-25203
- U15: symbol SMA -> fmcw3:SMA
- U7: footprint TO_SOT_Packages_SMD:SOT-353_SC-70-5 -> Package_TO_SOT_SMD:SOT-353_SC-70-5; symbol TLV172DCK -> fmcw3:TLV172DCK
- Z1: symbol BRANCHLINE -> fmcw3:BRANCHLINE
Connections:
- wire segments 158 -> 207
