File: hardware/usb.sch (KiCad schematic (older format))
At the start: 33 parts, among them U31 USB-MICRO, U32 93LC46B, U33 FT2232H, Y1 ABM10-167-12.000MHZ-T3

Commit message: Update kicad:  * kicad_pcb from 20170123 to 20171130 (pcbnew from 75cda50 to 5ecfd32)  * EESchema from 2 to 4
fix pin 53 in U33 (remove path in pcb)
Parts:
- C152, C153, C154, C155, C156, C157, C158, C159, C160, C161, C207, C208, C209, C210, C211, C212: symbol C -> Device:C
- FB12, FB14: symbol FILTER -> Device:L_Core_Ferrite
- R71, R72, R73, R79, R80, R81, R82, R83, R84, R85, R88: symbol R -> Device:R
- U31: symbol USB-MICRO -> fmcw3:USB-MICRO
- U32: symbol 93LC46B -> fmcw3:93LC46B
- U33: footprint Housings_QFP:LQFP-64_10x10mm_Pitch0.5mm -> Package_QFP:LQFP-64_10x10mm_P0.5mm; symbol FT2232H -> fmcw3:FT2232H
- Y1: symbol XTAL_SMD4 -> fmcw3:XTAL_SMD4
Connections:
- wire segments 108 -> 133
